File: RF_Schematic.sch (KiCad schematic (older format))
At the start: 0 parts

Commit message: First revision of RF circuit
Parts:
- added C?: 10u, symbol Device:C
- added C? (x4): 10n, symbol Device:C
- added C? (x6): 22p, symbol Device:C
- added C?: 220p, symbol Device:C
- added C?: 2u2, symbol Device:C
- added C?: 4p7, symbol Device:C
- added C?: 2n2, symbol Device:C
- added F1: 2450LP14B100, Low pass filter:2450BM14A0002, symbol Low~pass~filter:2450LP14B100
- added IC1: RFX2401C, RFX2401C:QFN50P300X300X60-17N-D, symbol RFX2401C:RFX2401C
- added J1: 5-1814400-1, SMA Connector 5-1814400-1 TE Connectivity:SMA_CONN_5-1814400-1, symbol 5-1814400-1:5-1814400-1
- added L?: 8n2, symbol Device:L
- added L?: 3n9, symbol Device:L
- added L?: 2n7, symbol Device:L
- added R?: 1M, symbol Device:R
- added R?: 22k, symbol Device:R
- added U1: nRF24L01P, Package_DFN_QFN:QFN-20-1EP_4x4mm_P0.5mm_EP2.5x2.5mm, symbol RF:nRF24L01P
- added Y?: 16MHz, symbol Device:Crystal_GND23_Small
Connections:
- net labels added: +3V3, GND, MISO, MOSI, NRF_ANT1, NRF_ANT2, NRF_CE, NRF_CS, NRF_IRQ, NRF_VDD_PA, NRF_XC1, NRF_XC2, RFX_ANT, RFX_TXRX, SCK
- wire segments 0 -> 149
Other:
- note added: "50 Ohm"
- note added: "Crystal oscilator"
- note added: "Filters for RFX"
- note added: "Filters for nRF"
- note added: "Impedance matching RFX -> Antenna"
- note added: "Impedance matching\nnRF24L01 -> RFX2401C"
- note added: "NRF24L01\nRadio"
- note added: "RF Amplifilier\nRFX2401C"
