File: RF_Schematic.sch (KiCad schematic (older format))
At the start: 25 parts, among them IC1 RFX2401C, J1 5-1814400-1, U1 nRF24L01P

Commit message: Little Corrections
Little corrections in RF circuit
Parts:
- gave numbers to parts that had none: 21
Connections:
- wire segments 149 -> 152
Other:
- note added: "Filters for RFX2401C"
- note added: "Filters for nRF24L01"
- note added: "Impedance matching RFX -> SMA Antenna"
- note added: "PLEASE VALIDATE THE CAPACITORS \nNEAR THE OSCILATOR !!!"
- note added: "nRF24L01\nRadio"
- note removed: "Filters for RFX"
- note removed: "Filters for nRF"
- note removed: "Impedance matching RFX -> Antenna"
- note removed: "NRF24L01\nRadio"
- moved on the sheet: C11, IC1, J1
